File: pcb/AutonomousCC/CC_PCB_V1.sch (KiCad schematic (older format))
At the start: 6 parts, among them J2 Antenna_Conn_02x04_Odd_Even, J3 USB1130-15-A_REVA, J5 Relay_Conn_01x06, U1 Pico, U2 level_converter_BOB-12009

Commit message: Updated
Parts:
- J2: symbol Connector_Generic:Conn_02x04_Odd_Even -> CC_PCB_V1-rescue:Conn_02x04_Odd_Even-Connector_Generic
- J5: symbol Connector_Generic:Conn_01x06 -> CC_PCB_V1-rescue:Conn_01x06-Connector_Generic
Changed lines of the file:
@@
 $EndComp
 $Comp
-L Connector_Generic:Conn_01x06 J5
+L CC_PCB_V1-rescue:Conn_01x06-Connector_Generic J5
 U 1 1 6132C346
 P 8620 5080
@@
 $EndComp
 $Comp
-L Connector_Generic:Conn_02x04_Odd_Even J2
+L CC_PCB_V1-rescue:Conn_02x04_Odd_Even-Connector_Generic J2
 U 1 1 6132E9AC
 P 9050 4000
@@
 $EndComp
 $Comp
-L power:GND #PWR0102
+L CC_PCB_V1-rescue:GND-power #PWR0102
 U 1 1 6139949D
 P 8400 3900
@@
 	7150 3750 7300 3750
 $Comp
-L power:GND #PWR0105
+L CC_PCB_V1-rescue:GND-power #PWR0105
 U 1 1 613C4FFD
 P 8020 4880
@@
 NoConn ~ 8420 5380
 $Comp
-L power:+5V #PWR0111
+L CC_PCB_V1-rescue:+5V-power #PWR0111
 U 1 1 6140F10C
 P 8170 5180
@@
 $EndComp
 $Comp
-L power:+5V #PWR0113
+L CC_PCB_V1-rescue:+5V-power #PWR0113
 U 1 1 614163BA
 P 8970 1840
@@
 NoConn ~ 8970 1740
 $Comp
-L power:GND #PWR0103
+L CC_PCB_V1-rescue:GND-power #PWR0103
 U 1 1 6132ADE6
 P 8970 1540
@@
 $EndComp
 $Comp
-L power:GND #PWR0101
+L CC_PCB_V1-rescue:GND-power #PWR0101
 U 1 1 6132D47F
 P 7470 2850
@@
 $EndComp
 $Comp
-L power:PWR_FLAG #FLG0103
+L CC_PCB_V1-rescue:PWR_FLAG-power #FLG0103
 U 1 1 6132C74E
 P 7150 2850
@@
 $EndComp
 $Comp
-L power:+5V #PWR0104
+L CC_PCB_V1-rescue:+5V-power #PWR0104
 U 1 1 613A9FB6
 P 5690 4450
@@
 NoConn ~ 5750 4150
 $Comp
-L power:PWR_FLAG #FLG0101
+L CC_PCB_V1-rescue:PWR_FLAG-power #FLG0101
 U 1 1 6138143E
 P 8970 1840
@@
 	5750 4450 5690 4450
 $Comp
-L power:+5V #PWR0106
+L CC_PCB_V1-rescue:+5V-power #PWR0106
 U 1 1 6137FAD9
 P 4600 1350
@@
 $EndComp
 $Comp
-L power:PWR_FLAG #FLG0105
+L CC_PCB_V1-rescue:PWR_FLAG-power #FLG0105
 U 1 1 61389C22
 P 4600 1350
@@
 $EndComp
 $Comp
-L power:GND #PWR0107
+L CC_PCB_V1-rescue:GND-power #PWR0107
 U 1 1 6138B5C9
 P 6000 2050
@@
 $EndComp
 $Comp
-L power:+5V #PWR0108
+L CC_PCB_V1-rescue:+5V-power #PWR0108
 U 1 1 6138D18B
 P 9450 3900
@@
 	6000 1350 6150 1350
 $Comp
-L power:GND #PWR0109
+L CC_PCB_V1-rescue:GND-power #PWR0109
 U 1 1 6139CFDB
 P 6150 1450
