File: pcb/AutonomousCC/Controller_V1/_autosave-Controller_V1.sch (KiCad schematic (older format))
At the start: 14 parts, among them J1 Antenna_Conn_02x04_Odd_Even, J2 USB1130-15-A_REVA, SW1 SW_12mm_Push, SW2 SW_12mm_Push, U1 COM-09032, U2 Pico, U3 COM-09032

Commit message: Updated pcb footprints
Parts:
- D1, D2: footprint (none) -> LED_THT:LED_D3.0mm
Connections:
- no-connect marks 41 -> 44
Changed lines of the file:
@@
 F 0 "D1" H 2293 6317 50  0000 C CNN
 F 1 "Green_LED" H 2293 6226 50  0000 C CNN
-F 2 "" H 2300 6100 50  0001 C CNN
+F 2 "LED_THT:LED_D3.0mm" H 2300 6100 50  0001 C CNN
 F 3 "~" H 2300 6100 50  0001 C CNN
 	1    2300 6100
@@
 F 0 "D2" H 4893 6317 50  0000 C CNN
 F 1 "RED_LED" H 4893 6226 50  0000 C CNN
-F 2 "" H 4900 6100 50  0001 C CNN
+F 2 "LED_THT:LED_D3.0mm" H 4900 6100 50  0001 C CNN
 F 3 "~" H 4900 6100 50  0001 C CNN
 	1    4900 6100
@@
 Wire Wire Line
 	4800 3550 4650 3550
+NoConn ~ 9000 5450
+NoConn ~ 9000 5550
+NoConn ~ 9000 5850
 $EndSCHEMATC
