File: pcb/AutonomousCC/CC_Brain_V1/CC_PCB_V1.kicad_pcb (KiCad board)
At the start: 2 copper layers, 104.2 x 144.9 mm, 37 parts, among them J1 Screw_Terminal_01x07, J2 Antenna_Conn_02x04_Odd_Even, J3 USB1130-15-A_REVA, J4 Conn_01x02_Male, J5 Relay_Conn_01x06, J6 Conn_01x02_Male, J7 Linear Actuator Power, J8 Linear Actuator, J9 Conn_01x02_Male, K1 FINDER-40.11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

Commit message: Saved Gerber Files
Other:
- board text added: "Autonomous Crazy Cart V2"
- board text added: "Design by: Dylan Ballback, Jacob Romeo, Daniel Wilczak"
- board text removed: "Autonomous Crazy Cart V1.1"
- board text removed: "Design by: Jacob Romeo, Daniel Wilczak, Dylan Ballback"
Changed lines of the file:
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@@
-(kicad_pcb (version 20171130) (host pcbnew "(5.1.10)-1")
+(kicad_pcb (version 20171130) (host pcbnew "(5.1.10-1-10_14)")
   (general
     (thickness 1.6)
@@
       (effects (font (size 1 1) (thickness 0.15)) (justify mirror))
     )
-    (fp_text user %R (at 0 0 270) (layer B.Fab)
-      (effects (font (size 0.4 0.4) (thickness 0.06)) (justify mirror))
-    )
     (fp_line (start -0.8 -0.4125) (end -0.8 0.4125) (layer B.Fab) (width 0.1))
     (fp_line (start -0.8 0.4125) (end 0.8 0.4125) (layer B.Fab) (width 0.1))
@@
     (fp_line (start 1.65 0.73) (end 1.65 -0.73) (layer B.CrtYd) (width 0.05))
     (fp_line (start 1.65 -0.73) (end -1.65 -0.73) (layer B.CrtYd) (width 0.05))
+    (fp_text user %R (at 0 0 270) (layer B.Fab)
+      (effects (font (size 0.4 0.4) (thickness 0.06)) (justify mirror))
+    )
     (pad 2 smd roundrect (at 0.9125 0 270) (size 0.975 0.95) (layers B.Cu B.Paste B.Mask) (roundrect_rratio 0.25)
       (net 40 GP12))
@@
     (fp_text value 1k (at 0 -1.43 -90) (layer B.Fab)
       (effects (font (size 1 1) (thickness 0.15)) (justify mirror))
-    )
-    (fp_text user %R (at 0 0 -90) (layer B.Fab) hide
-      (effects (font (size 0.4 0.4) (thickness 0.06)) (justify mirror))
     )
     (fp_line (start -0.8 -0.4125) (end -0.8 0.4125) (layer B.Fab) (width 0.1))
@@
     (fp_line (start 1.65 0.73) (end 1.65 -0.73) (layer B.CrtYd) (width 0.05))
     (fp_line (start 1.65 -0.73) (end -1.65 -0.73) (layer B.CrtYd) (width 0.05))
+    (fp_text user %R (at 0 0 -90) (layer B.Fab) hide
+      (effects (font (size 0.4 0.4) (thickness 0.06)) (justify mirror))
+    )
     (pad 2 smd roundrect (at 0.9125 0 90) (size 0.975 0.95) (layers B.Cu B.Paste B.Mask) (roundrect_rratio 0.25)
       (net 37 GP22))
@@
     (fp_text value "SMD LED2" (at 0 1.82 90) (layer F.Fab)
       (effects (font (size 1 1) (thickness 0.15)))
-    )
-    (fp_text user %R (at 0 0 90) (layer F.Fab)
-      (effects (font (size 0.8 0.8) (thickness 0.12)))
     )
     (fp_line (start 1.6 -0.8) (end -1.2 -0.8) (layer F.Fab) (width 0.1))
@@
     (fp_line (start 2.45 -1.12) (end 2.45 1.12) (layer F.CrtYd) (width 0.05))
     (fp_line (start 2.45 1.12) (end -2.45 1.12) (layer F.CrtYd) (width 0.05))
-    (pad 2 smd roundrect (at 1.4875 0 90) (size 1.425 1.75) (layers F.Cu F.Paste F.Mask) (roundrect_rratio 0.175439)
+    (fp_text user %R (at 0 0 90) (layer F.Fab)
+      (effects (font (size 0.8 0.8) (thickness 0.12)))
+    )
+    (pad 2 smd roundrect (at 1.4875 0 90) (size 1.425 1.75) (layers F.Cu F.Paste F.Mask) (roundrect_rratio 0.1754385964912281)
       (net 70 "Net-(D6-Pad2)"))
-    (pad 1 smd roundrect (at -1.4875 0 90) (size 1.425 1.75) (layers F.Cu F.Paste F.Mask) (roundrect_rratio 0.175439)
+    (pad 1 smd roundrect (at -1.4875 0 90) (size 1.425 1.75) (layers F.Cu F.Paste F.Mask) (roundrect_rratio 0.1754385964912281)
       (net 71 "Net-(D6-Pad1)"))
     (model ${KISYS3DMOD}/LED_SMD.3dshapes/LED_1206_3216Metric.wrl
@@
     (fp_text value "SMD LED2" (at 0 1.82 90) (layer F.Fab)
       (effects (font (size 1 1) (thickness 0.15)))
-    )
-    (fp_text user %R (at 0 0 90) (layer F.Fab)
-      (effects (font (size 0.8 0.8) (thickness 0.12)))
     )
     (fp_line (start 1.6 -0.8) (end -1.2 -0.8) (layer F.Fab) (width 0.1))
@@
     (fp_line (start 2.45 -1.12) (end 2.45 1.12) (layer F.CrtYd) (width 0.05))
     (fp_line (start 2.45 1.12) (end -2.45 1.12) (layer F.CrtYd) (width 0.05))
-    (pad 2 smd roundrect (at 1.4875 0 90) (size 1.425 1.75) (layers F.Cu F.Paste F.Mask) (roundrect_rratio 0.175439)
+    (fp_text user %R (at 0 0 90) (layer F.Fab)
+      (effects (font (size 0.8 0.8) (thickness 0.12)))
+    )
+    (pad 2 smd roundrect (at 1.4875 0 90) (size 1.425 1.75) (layers F.Cu F.Paste F.Mask) (roundrect_rratio 0.1754385964912281)
       (net 68 "Net-(D5-Pad2)"))
-    (pad 1 smd roundrect (at -1.4875 0 90) (size 1.425 1.75) (layers F.Cu F.Paste F.Mask) (roundrect_rratio 0.175439)
+    (pad 1 smd roundrect (at -1.4875 0 90) (size 1.425 1.75) (layers F.Cu F.Paste F.Mask) (roundrect_rratio 0.1754385964912281)
       (net 69 "Net-(D5-Pad1)"))
     (model ${KISYS3DMOD}/LED_SMD.3dshapes/LED_1206_3216Metric.wrl
@@
       (effects (font (size 0.8 0.8) (thickness 0.12)))
     )
-    (pad 2 smd roundrect (at 1.4875 0 90) (size 1.425 2.65) (layers F.Cu F.Paste F.Mask) (roundrect_rratio 0.175439)
+    (pad 2 smd roundrect (at 1.4875 0 90) (size 1.425 2.65) (layers F.Cu F.Paste F.Mask) (roundrect_rratio 0.1754385964912281)
       (net 53 "Net-(D4-Pad2)"))
-    (pad 1 smd roundrect (at -1.4875 0 90) (size 1.425 2.65) (layers F.Cu F.Paste F.Mask) (roundrect_rratio 0.175439)
+    (pad 1 smd roundrect (at -1.4875 0 90) (size 1.425 2.65) (layers F.Cu F.Paste F.Mask) (roundrect_rratio 0.1754385964912281)
       (net 59 "Net-(D4-Pad1)"))
     (model ${KISYS3DMOD}/Diode_SMD.3dshapes/D_1210_3225Metric.wrl
@@
       (effects (font (size 0.8 0.8) (thickness 0.12)))
     )
-    (pad 2 smd roundrect (at 1.4875 0 90) (size 1.425 2.65) (layers F.Cu F.Paste F.Mask) (roundrect_rratio 0.175439)
+    (pad 2 smd roundrect (at 1.4875 0 90) (size 1.425 2.65) (layers F.Cu F.Paste F.Mask) (roundrect_rratio 0.1754385964912281)
       (net 52 "Net-(D3-Pad2)"))
-    (pad 1 smd roundrect (at -1.4875 0 90) (size 1.425 2.65) (layers F.Cu F.Paste F.Mask) (roundrect_rratio 0.175439)
+    (pad 1 smd roundrect (at -1.4875 0 90) (size 1.425 2.65) (layers F.Cu F.Paste F.Mask) (roundrect_rratio 0.1754385964912281)
       (net 58 "Net-(D3-Pad1)"))
     (model ${KISYS3DMOD}/Diode_SMD.3dshapes/D_1210_3225Metric.wrl
@@
       (effects (font (size 0.8 0.8) (thickness 0.12)))
     )
-    (pad 2 smd roundrect (at 1.4875 0 90) (size 1.425 1.75) (layers F.Cu F.Paste F.Mask) (roundrect_rratio 0.175439)
+    (pad 2 smd roundrect (at 1.4875 0 90) (size 1.425 1.75) (layers F.Cu F.Paste F.Mask) (roundrect_rratio 0.1754385964912281)
       (net 64 "Net-(D2-Pad2)"))
-    (pad 1 smd roundrect (at -1.4875 0 90) (size 1.425 1.75) (layers F.Cu F.Paste F.Mask) (roundrect_rratio 0.175439)
+    (pad 1 smd roundrect (at -1.4875 0 90) (size 1.425 1.75) (layers F.Cu F.Paste F.Mask) (roundrect_rratio 0.1754385964912281)
       (net 44 GP11))
     (model ${KISYS3DMOD}/LED_SMD.3dshapes/LED_1206_3216Metric.wrl
@@
       (effects (font (size 0.8 0.8) (thickness 0.12)))
     )
-    (pad 2 smd roundrect (at 1.4875 0 90) (size 1.425 1.75) (layers F.Cu F.Paste F.Mask) (roundrect_rratio 0.175439)
+    (pad 2 smd roundrect (at 1.4875 0 90) (size 1.425 1.75) (layers F.Cu F.Paste F.Mask) (roundrect_rratio 0.1754385964912281)
       (net 61 "Net-(D1-Pad2)"))
-    (pad 1 smd roundrect (at -1.4875 0 90) (size 1.425 1.75) (layers F.Cu F.Paste F.Mask) (roundrect_rratio 0.175439)
+    (pad 1 smd roundrect (at -1.4875 0 90) (size 1.425 1.75) (layers F.Cu F.Paste F.Mask) (roundrect_rratio 0.1754385964912281)
       (net 45 GP10))
     (model ${KISYS3DMOD}/LED_SMD.3dshapes/LED_1206_3216Metric.wrl
@@
   (gr_line (start 158.801286 21.953499) (end 158.653499 156.1) (layer Edge.Cuts) (width 0.5))
   (gr_line (start 60.053499 16.498714) (end 153.6 16.5) (layer Edge.Cuts) (width 0.5))
-  (gr_text "Design by: Jacob Romeo, Daniel Wilczak, Dylan Ballback" (at 115 18.4) (layer F.Mask)
+  (gr_text "Design by: Dylan Ballback, Jacob Romeo, Daniel Wilczak " (at 115 18.4) (layer F.Mask)
     (effects (font (size 1.5 1.5) (thickness 0.3)))
   )
-  (gr_text "Autonomous Crazy Cart V1.1\n\n" (at 123.9901 160.2613) (layer F.Mask)
+  (gr_text "Autonomous Crazy Cart V2\n\n" (at 122.2375 160.909) (layer F.Mask)
     (effects (font (size 3 3) (thickness 0.5)))
   )

Commit message: CC Controller and Brain VERSION 1.1
Parts:
- removed Re: 1k, Resistor_SMD:R_0603_1608Metric_Pad0.98x0.95mm_HandSolder
- removed THROTTLE: SMD LED2, LED_SMD:LED_1206_3216Metric_Pad1.42x1.75mm_HandSolder
- added D5: SMD LED2, LED_SMD:LED_1206_3216Metric_Pad1.42x1.75mm_HandSolder, F.Cu at (138.6, 128.9)
- added R5: 1k, Resistor_SMD:R_0603_1608Metric_Pad0.98x0.95mm_HandSolder, F.Cu at (137.1, 124.4)
- R6: moved to F.Cu
- moved R6 10.6 mm to (137.1, 115.6), turned to 90 degrees
- moved D6 2.20 mm to (138.6, 120.5), turned to 180 degrees
- renumbered STEP to D6
Connections:
- D6 pad 1: Net-(D6-Pad1) -> GND
Routing:
- net GP26: track 77.0 -> 89.3 mm
- net Net-(D6-Pad2): track 13.0 -> 3.94 mm, vias 1 -> 0
- net Net-(D5-Pad2): track 10.3 -> 3.57 mm, vias 1 -> 0
- net GP22: track 77.6 -> 83.6 mm, vias 0 -> 2
- net GND: track 44.3 -> 39.2 mm, vias 9 -> 7
- net GP12: track 64.5 -> 68.5 mm, vias 0 -> 1
Other:
- board text added: "Autonomous Crazy Cart V1.1"
- board text removed: "Autonomous Crazy Cart V2"
