File: pcb/AutonomousCC/CC_Brain_V1/relay.sch (KiCad schematic (older format))
At the start: 18 parts, among them J4 Conn_01x02_Male, J6 Conn_01x02_Male, J7 Linear Actuator Power, J8 Linear Actuator, K1 FINDER-40.11, K2 FINDER-40.11, Q1 PC817A, Q2 PC817A, Q3 BC547A, Q4 BC547A

Commit message: Added most of the footprints
Still need Diodes, Resistors (if THT or SMD), and LED footprints
Parts:
- J4, J6: footprint (none) -> Connector_PinHeader_2.54mm:PinHeader_1x02_P2.54mm_Vertical
- J7, J8: footprint (none) -> MCU_RaspberryPi_and_Boards:TE_282837-2
- Q1, Q2: footprint DIP762W50P254L650H458Q4B -> MCU_RaspberryPi_and_Boards:DIP762W50P254L650H458Q4B
Changed lines of the file:
@@
 F 0 "Q1" H 4350 2897 50  0000 C CNN
 F 1 "PC817A" H 4350 2806 50  0000 C CNN
-F 2 "DIP762W50P254L650H458Q4B" H 4350 2550 50  0001 L BNN
+F 2 "MCU_RaspberryPi_and_Boards:DIP762W50P254L650H458Q4B" H 4350 2550 50  0001 L BNN
 F 3 "" H 4350 2550 50  0001 L BNN
 F 4 "PC817A" H 4350 2550 50  0001 L BNN "MP"
@@
 F 0 "J4" V 4550 1400 50  0000 L CNN
 F 1 "Conn_01x02_Male" V 4650 1400 50  0000 L CNN
-F 2 "" H 4600 1350 50  0001 C CNN
+F 2 "Connector_PinHeader_2.54mm:PinHeader_1x02_P2.54mm_Vertical" H 4600 1350 50  0001 C CNN
 F 3 "~" H 4600 1350 50  0001 C CNN
 	1    4600 1350
@@
 F 0 "Q2" H 4350 5697 50  0000 C CNN
 F 1 "PC817A" H 4350 5606 50  0000 C CNN
-F 2 "DIP762W50P254L650H458Q4B" H 4350 5350 50  0001 L BNN
+F 2 "MCU_RaspberryPi_and_Boards:DIP762W50P254L650H458Q4B" H 4350 5350 50  0001 L BNN
 F 3 "" H 4350 5350 50  0001 L BNN
 F 4 "PC817A" H 4350 5350 50  0001 L BNN "MP"
@@
 F 0 "J6" V 4550 4200 50  0000 L CNN
 F 1 "Conn_01x02_Male" V 4650 4200 50  0000 L CNN
-F 2 "" H 4600 4150 50  0001 C CNN
+F 2 "Connector_PinHeader_2.54mm:PinHeader_1x02_P2.54mm_Vertical" H 4600 4150 50  0001 C CNN
 F 3 "~" H 4600 4150 50  0001 C CNN
 	1    4600 4150
@@
 F 0 "J8" H 9980 3292 50  0000 L CNN
 F 1 "Linear Actuator" H 9980 3201 50  0000 L CNN
-F 2 "" H 9900 3300 50  0001 C CNN
+F 2 "MCU_RaspberryPi_and_Boards:TE_282837-2" H 9900 3300 50  0001 C CNN
 F 3 "~" H 9900 3300 50  0001 C CNN
 	1    9900 3300
@@
 F 0 "J7" H 9980 2842 50  0000 L CNN
 F 1 "Linear Actuator Power" H 9980 2751 50  0000 L CNN
-F 2 "" H 9900 2850 50  0001 C CNN
+F 2 "MCU_RaspberryPi_and_Boards:TE_282837-2" H 9900 2850 50  0001 C CNN
 F 3 "~" H 9900 2850 50  0001 C CNN
 	1    9900 2850

Commit message: Updated Footprints and PCB Layout
Parts:
- D1: value SMD LED -> SMD LED1; footprint (none) -> LED_SMD:LED_1206_3216Metric_Pad1.42x1.75mm_HandSolder
- D2: value SMD LED -> SMD LED2; footprint (none) -> LED_SMD:LED_1206_3216Metric_Pad1.42x1.75mm_HandSolder
- D3, D4: footprint (none) -> Diode_SMD:D_1210_3225Metric_Pad1.42x2.65mm_HandSolder
- K1, K2: footprint Relay_THT:Relay_SPDT_Finder_40.11 -> Relay_THT:Relay_SPDT_Finder_36.11
- R1, R2, R3, R4: footprint (none) -> Resistor_SMD:R_0603_1608Metric_Pad0.98x0.95mm_HandSolder
Changed lines of the file:
@@
 F 0 "K1" H 7180 1996 50  0000 L CNN
 F 1 "FINDER-40.11" H 7180 1905 50  0000 L CNN
-F 2 "Relay_THT:Relay_SPDT_Finder_40.11" H 7890 1910 50  0001 C CNN
+F 2 "Relay_THT:Relay_SPDT_Finder_36.11" H 7890 1910 50  0001 C CNN
 F 3 "https://www.finder-relais.net/de/finder-relais-serie-40.pdf" H 6750 1950 50  0001 C CNN
 	1    6750 1950
@@
 F 0 "D3" V 5946 1822 50  0000 R CNN
 F 1 "DIODE" V 5855 1822 50  0000 R CNN
-F 2 "" H 5900 1950 50  0001 C CNN
+F 2 "Diode_SMD:D_1210_3225Metric_Pad1.42x2.65mm_HandSolder" H 5900 1950 50  0001 C CNN
 F 3 "~" H 5900 1950 50  0001 C CNN
 	1    5900 1950
@@
 F 0 "R3" V 4945 2650 50  0000 C CNN
 F 1 "1k" V 5036 2650 50  0000 C CNN
-F 2 "" H 5150 2650 50  0001 C CNN
+F 2 "Resistor_SMD:R_0603_1608Metric_Pad0.98x0.95mm_HandSolder" H 5150 2650 50  0001 C CNN
 F 3 "~" H 5150 2650 50  0001 C CNN
 	1    5150 2650
@@
 F 0 "R1" H 4018 1996 50  0000 L CNN
 F 1 "1k" H 4018 1905 50  0000 L CNN
-F 2 "" H 3950 1950 50  0001 C CNN
+F 2 "Resistor_SMD:R_0603_1608Metric_Pad0.98x0.95mm_HandSolder" H 3950 1950 50  0001 C CNN
 F 3 "~" H 3950 1950 50  0001 C CNN
 	1    3950 1950
@@
 P 3600 2650
 F 0 "D1" H 3593 2867 50  0000 C CNN
-F 1 "SMD LED" H 3593 2776 50  0000 C CNN
-F 2 "" H 3600 2650 50  0001 C CNN
+F 1 "SMD LED1" H 3593 2776 50  0000 C CNN
+F 2 "LED_SMD:LED_1206_3216Metric_Pad1.42x1.75mm_HandSolder" H 3600 2650 50  0001 C CNN
 F 3 "~" H 3600 2650 50  0001 C CNN
 	1    3600 2650
@@
 F 0 "K2" H 7180 4796 50  0000 L CNN
 F 1 "FINDER-40.11" H 7180 4705 50  0000 L CNN
-F 2 "Relay_THT:Relay_SPDT_Finder_40.11" H 7890 4710 50  0001 C CNN
+F 2 "Relay_THT:Relay_SPDT_Finder_36.11" H 7890 4710 50  0001 C CNN
 F 3 "https://www.finder-relais.net/de/finder-relais-serie-40.pdf" H 6750 4750 50  0001 C CNN
 	1    6750 4750
@@
 F 0 "D4" V 5946 4622 50  0000 R CNN
 F 1 "DIODE" V 5855 4622 50  0000 R CNN
-F 2 "" H 5900 4750 50  0001 C CNN
+F 2 "Diode_SMD:D_1210_3225Metric_Pad1.42x2.65mm_HandSolder" H 5900 4750 50  0001 C CNN
 F 3 "~" H 5900 4750 50  0001 C CNN
 	1    5900 4750
@@
 F 0 "R4" V 4945 5450 50  0000 C CNN
 F 1 "1k" V 5036 5450 50  0000 C CNN
-F 2 "" H 5150 5450 50  0001 C CNN
+F 2 "Resistor_SMD:R_0603_1608Metric_Pad0.98x0.95mm_HandSolder" H 5150 5450 50  0001 C CNN
 F 3 "~" H 5150 5450 50  0001 C CNN
 	1    5150 5450
@@
 F 0 "R2" H 4018 4796 50  0000 L CNN
 F 1 "1k" H 4018 4705 50  0000 L CNN
-F 2 "" H 3950 4750 50  0001 C CNN
+F 2 "Resistor_SMD:R_0603_1608Metric_Pad0.98x0.95mm_HandSolder" H 3950 4750 50  0001 C CNN
 F 3 "~" H 3950 4750 50  0001 C CNN
 	1    3950 4750
@@
 P 3600 5450
 F 0 "D2" H 3593 5667 50  0000 C CNN
-F 1 "SMD LED" H 3593 5576 50  0000 C CNN
-F 2 "" H 3600 5450 50  0001 C CNN
+F 1 "SMD LED2" H 3593 5576 50  0000 C CNN
+F 2 "LED_SMD:LED_1206_3216Metric_Pad1.42x1.75mm_HandSolder" H 3600 5450 50  0001 C CNN
 F 3 "~" H 3600 5450 50  0001 C CNN
 	1    3600 5450
