File: pcb/Linear_Actuator_PCB/Linear_Actuator_PCB.kicad_sch (KiCad schematic)
At the start: 27 parts, among them J1 Pwr/Coms, J2 Pot, J3 Bootloader Pins, J5 LED, J7 8P8C, SW1 SW_Push, U1 ATmega328P-AU, Y1 Crystal

Commit message: Finished tracing the Linear Actuator
Other:
- sheet relay renamed RELAY
- sheet RELAY ports: added Relay1, Relay2; removed none
- moved on the sheet: J7
Changed lines of the file:
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@@
     (stroke (width 0) (type default) (color 0 0 0 0))
   )
-  (wire (pts (xy 106.553 163.449) (xy 115.57 163.449))
+  (wire (pts (xy 106.553 163.83) (xy 115.57 163.83))
     (stroke (width 0) (type default) (color 0 0 0 0))
   )
@@
     (effects (font (size 1.27 1.27)) (justify right bottom))
   )
-  (label "SCL" (at 264.795 48.26 180)
+  (label "SCL" (at 259.08 48.26 180)
     (effects (font (size 1.27 1.27)) (justify right bottom))
   )
@@
     (effects (font (size 1.27 1.27)) (justify right bottom))
   )
-  (label "relay2" (at 79.375 130.175 180)
+  (label "Relay2" (at 79.375 130.175 180)
     (effects (font (size 1.27 1.27)) (justify right bottom))
   )
@@
     (effects (font (size 1.27 1.27)) (justify left bottom))
   )
-  (label "relay1" (at 106.553 163.449 0)
+  (label "Relay1" (at 106.553 163.83 0)
     (effects (font (size 1.27 1.27)) (justify left bottom))
   )
@@
     (effects (font (size 1.27 1.27)) (justify right bottom))
   )
-  (label "RXD" (at 264.795 53.34 180)
+  (label "RXD" (at 259.08 53.34 180)
     (effects (font (size 1.27 1.27)) (justify right bottom))
   )
@@
     (effects (font (size 1.27 1.27)) (justify left bottom))
   )
-  (label "TXD" (at 264.795 55.88 180)
-    (effects (font (size 1.27 1.27)) (justify right bottom))
-  )
-  (label "relay1" (at 79.375 127.635 180)
-    (effects (font (size 1.27 1.27)) (justify right bottom))
-  )
-  (label "relay2" (at 106.553 167.64 0)
+  (label "TXD" (at 259.08 55.88 180)
+    (effects (font (size 1.27 1.27)) (justify right bottom))
+  )
+  (label "Relay1" (at 79.375 127.635 180)
+    (effects (font (size 1.27 1.27)) (justify right bottom))
+  )
+  (label "Relay2" (at 106.553 167.64 0)
     (effects (font (size 1.27 1.27)) (justify left bottom))
   )
@@
     (effects (font (size 1.27 1.27)) (justify right bottom))
   )
-  (label "SDA" (at 264.795 50.8 180)
+  (label "SDA" (at 259.08 50.8 180)
     (effects (font (size 1.27 1.27)) (justify right bottom))
   )
@@
   (label "SDA" (at 74.93 109.855 180)
     (effects (font (size 1.27 1.27)) (justify right bottom))
-  )
-  (hierarchical_label "Relay1" (shape input) (at 115.57 163.449 0)
-    (effects (font (size 1.27 1.27)) (justify left))
-  )
-  (hierarchical_label "Relay2" (shape input) (at 115.57 167.64 0)
-    (effects (font (size 1.27 1.27)) (justify left))
   )
   (symbol (lib_id "MCU_Microchip_ATmega:ATmega328P-AU") (at 52.705 107.315 0) (unit 1)
@@
     (pin "1")
   )
-  (symbol (lib_id "power:GND") (at 264.795 40.64 270) (unit 1)
+  (symbol (lib_id "power:GND") (at 259.08 40.64 270) (unit 1)
     (in_bom yes) (on_board yes) (fields_autoplaced)
-    (property "Reference" "#PWR0133" (id 0) (at 258.445 40.64 0)
-      (effects (font (size 1.27 1.27)) hide)
-    )
-    (property "Value" "GND" (id 1) (at 261.6201 41.0738 90)
-      (effects (font (size 1.27 1.27)) (justify right))
-    )
-    (property "Footprint" "" (id 2) (at 264.795 40.64 0)
-      (effects (font (size 1.27 1.27)) hide)
-    )
-    (property "Datasheet" "" (id 3) (at 264.795 40.64 0)
+    (property "Reference" "#PWR0133" (id 0) (at 252.73 40.64 0)
+      (effects (font (size 1.27 1.27)) hide)
+    )
+    (property "Value" "GND" (id 1) (at 255.9051 41.0738 90)
+      (effects (font (size 1.27 1.27)) (justify right))
+    )
+    (property "Footprint" "" (id 2) (at 259.08 40.64 0)
+      (effects (font (size 1.27 1.27)) hide)
+    )
+    (property "Datasheet" "" (id 3) (at 259.08 40.64 0)
       (effects (font (size 1.27 1.27)) hide)
     )
@@
     (pin "1")
   )
-  (symbol (lib_id "power:GND") (at 264.795 38.1 270) (unit 1)
+  (symbol (lib_id "power:GND") (at 259.08 38.1 270) (unit 1)
     (in_bom yes) (on_board yes) (fields_autoplaced)
-    (property "Reference" "#PWR0128" (id 0) (at 258.445 38.1 0)
-      (effects (font (size 1.27 1.27)) hide)
-    )
-    (property "Value" "GND" (id 1) (at 261.6201 38.5338 90)
-      (effects (font (size 1.27 1.27)) (justify right))
-    )
-    (property "Footprint" "" (id 2) (at 264.795 38.1 0)
-      (effects (font (size 1.27 1.27)) hide)
-    )
-    (property "Datasheet" "" (id 3) (at 264.795 38.1 0)
+    (property "Reference" "#PWR0128" (id 0) (at 252.73 38.1 0)
+      (effects (font (size 1.27 1.27)) hide)
+    )
+    (property "Value" "GND" (id 1) (at 255.9051 38.5338 90)
+      (effects (font (size 1.27 1.27)) (justify right))
+    )
+    (property "Footprint" "" (id 2) (at 259.08 38.1 0)
+      (effects (font (size 1.27 1.27)) hide)
+    )
+    (property "Datasheet" "" (id 3) (at 259.08 38.1 0)
       (effects (font (size 1.27 1.27)) hide)
     )
@@
     (pin "1")
   )
-  (symbol (lib_id "Connector:8P8C") (at 274.955 45.72 180) (unit 1)
+  (symbol (lib_id "Connector:8P8C") (at 269.24 45.72 180) (unit 1)
     (in_bom yes) (on_board yes) (fields_autoplaced)
-    (property "Reference" "J7" (id 0) (at 283.337 46.1553 0)
-      (effects (font (size 1.27 1.27)) (justify right))
-    )
-    (property "Value" "8P8C" (id 1) (at 283.337 48.6922 0)
-      (effects (font (size 1.27 1.27)) (justify right))
-    )
-    (property "Footprint" "Connector_RJ:RJ45_Ninigi_GE" (id 2) (at 274.955 46.355 90)
-      (effects (font (size 1.27 1.27)) hide)
-    )
-    (property "Datasheet" "~" (id 3) (at 274.955 46.355 90)
+    (property "Reference" "J7" (id 0) (at 277.622 46.1553 0)
+      (effects (font (size 1.27 1.27)) (justify right))
+    )
+    (property "Value" "8P8C" (id 1) (at 277.622 48.6922 0)
+      (effects (font (size 1.27 1.27)) (justify right))
+    )
+    (property "Footprint" "Connector_RJ:RJ45_Ninigi_GE" (id 2) (at 269.24 46.355 90)
+      (effects (font (size 1.27 1.27)) hide)
+    )
+    (property "Datasheet" "~" (id 3) (at 269.24 46.355 90)
       (effects (font (size 1.27 1.27)) hide)
     )
@@
     (pin "3")
   )
-  (symbol (lib_id "power:+12V") (at 264.795 43.18 90) (unit 1)
+  (symbol (lib_id "power:+12V") (at 259.08 43.18 90) (unit 1)
     (in_bom yes) (on_board yes) (fields_autoplaced)
-    (property "Reference" "#PWR0134" (id 0) (at 268.605 43.18 0)
-      (effects (font (size 1.27 1.27)) hide)
-    )
-    (property "Value" "+12V" (id 1) (at 261.62 43.6138 90)
-      (effects (font (size 1.27 1.27)) (justify left))
-    )
-    (property "Footprint" "" (id 2) (at 264.795 43.18 0)
-      (effects (font (size 1.27 1.27)) hide)
-    )
-    (property "Datasheet" "" (id 3) (at 264.795 43.18 0)
+    (property "Reference" "#PWR0134" (id 0) (at 262.89 43.18 0)
+      (effects (font (size 1.27 1.27)) hide)
+    )
+    (property "Value" "+12V" (id 1) (at 255.905 43.6138 90)
+      (effects (font (size 1.27 1.27)) (justify left))
+    )
+    (property "Footprint" "" (id 2) (at 259.08 43.18 0)
+      (effects (font (size 1.27 1.27)) hide)
+    )
+    (property "Datasheet" "" (id 3) (at 259.08 43.18 0)
       (effects (font (size 1.27 1.27)) hide)
     )
@@
     (pin "6")
   )
-  (symbol (lib_id "power:+12V") (at 264.795 45.72 90) (unit 1)
+  (symbol (lib_id "power:+12V") (at 259.08 45.72 90) (unit 1)
     (in_bom yes) (on_board yes) (fields_autoplaced)
-    (property "Reference" "#PWR0127" (id 0) (at 268.605 45.72 0)
-      (effects (font (size 1.27 1.27)) hide)
-    )
-    (property "Value" "+12V" (id 1) (at 261.62 46.1538 90)
-      (effects (font (size 1.27 1.27)) (justify left))
-    )
-    (property "Footprint" "" (id 2) (at 264.795 45.72 0)
-      (effects (font (size 1.27 1.27)) hide)
-    )
-    (property "Datasheet" "" (id 3) (at 264.795 45.72 0)
+    (property "Reference" "#PWR0127" (id 0) (at 262.89 45.72 0)
+      (effects (font (size 1.27 1.27)) hide)
+    )
+    (property "Value" "+12V" (id 1) (at 255.905 46.1538 90)
+      (effects (font (size 1.27 1.27)) (justify left))
+    )
+    (property "Footprint" "" (id 2) (at 259.08 45.72 0)
+      (effects (font (size 1.27 1.27)) hide)
+    )
+    (property "Datasheet" "" (id 3) (at 259.08 45.72 0)
       (effects (font (size 1.27 1.27)) hide)
     )
@@
     (stroke (width 0.1524) (type solid) (color 0 0 0 0))
     (fill (color 0 0 0 0.0000))
-    (property "Sheet name" "relay" (id 0) (at 115.57 153.5934 0)
+    (property "Sheet name" "RELAY" (id 0) (at 115.57 153.5934 0)
       (effects (font (size 1.27 1.27)) (justify left bottom))
     )
@@
       (effects (font (size 1.27 1.27)) (justify left top))
     )
-  )
+    (pin "Relay2" input (at 115.57 167.64 180)
+      (effects (font (size 1.27 1.27)) (justify left))
+    )
+    (pin "Relay1" input (at 115.57 163.83 180)
+      (effects (font (size 1.27 1.27)) (justify left))
+    )
+  )
