File: pcb/Main_Controller_PCB V0.1/Main_Controller_PCB V0.1.kicad_pcb (KiCad board)
At the start: 2 copper layers, 75.9 x 57.4 mm, 16 parts, among them J1 Pwr/Coms, J2 Pwr/Coms, J3 LED, J4 Foot Pedal, J5 Pedal PWM, J6 Screw_Terminal_01x02, J7 8P8C, J8 8P8C

Commit message: Finished Traces
Routing:
- net GND: track 0.00 -> 177.3 mm, vias 0 -> 3
- net +12V: track 0.00 -> 121.9 mm, vias 0 -> 2
- net /SCL: track 0.00 -> 104.5 mm, vias 0 -> 3
- net /SDA: track 0.00 -> 98.1 mm, vias 0 -> 2
- net /TXD: track 0.00 -> 79.0 mm, vias 0 -> 4
- net /RXD: track 0.00 -> 75.6 mm, vias 0 -> 1
- net +5V: track 0.00 -> 59.7 mm, vias 0 -> 4
- net /LED: track 0.00 -> 39.1 mm, vias 0 -> 1
- net /pedal_pwm: track 0.00 -> 35.1 mm
- net /pedal: track 0.00 -> 23.0 mm, vias 0 -> 1

Commit message: Updated
Routing:
- net GND: track 177.3 -> 189.9 mm, vias 3 -> 2
- net +5V: track 59.7 -> 63.4 mm, vias 4 -> 3
- net +12V: track 121.9 -> 118.5 mm
- net /SDA: track 98.1 -> 98.0 mm, vias 2 -> 1
Other:
- outline, holes or cut-outs redrawn

Commit message: Uploaded Gerber
Routing:
- net GND: track 189.9 -> 186.3 mm, vias 2 -> 1
- net /SDA: track 98.0 -> 98.1 mm, vias 1 -> 0
- net /TXD: track 79.0 -> 78.9 mm, vias 4 -> 2
- net /SCL: vias 3 -> 2
- net /RXD: vias 1 -> 0
