File: pcb/Linear_Actuator_PCB V0.1/Linear_Actuator_PCB.kicad_sch (KiCad schematic)
At the start: 28 parts, among them J1 Pwr/Coms, J2 Pot, J3 Bootloader Pins, J5 LED, J7 8P8C, SW1 SW_Push, U1 ATmega328P-AU, Y1 Crystal

Commit message: New RC control PCB for dirft cart
Parts:
- removed C1, C2, C6, C8: 100nF, Capacitor_SMD:C_0603_1608Metric, symbol Device:C_Small
- removed C3, C4: 22pf, Capacitor_SMD:C_0603_1608Metric, symbol Device:C_Small
- removed C5: 0.33 uF, Capacitor_SMD:C_0603_1608Metric, symbol Device:C
- removed C7: 0.1uF, Capacitor_SMD:C_0603_1608Metric, symbol Device:CP1_Small
- removed J1: Pwr/Coms, Connector_PinHeader_2.54mm:PinHeader_1x06_P2.54mm_Vertical, symbol Connector:Conn_01x06_Female
- removed J3: Bootloader Pins, Connector_PinHeader_2.54mm:PinHeader_2x03_P2.54mm_Vertical, symbol Connector_Generic:Conn_02x03_Odd_Even
- removed J7: 8P8C, Connector_RJ:RJ45_Ninigi_GE, symbol Connector:8P8C
- removed R5: 10k, Resistor_SMD:R_0805_2012Metric, symbol Device:R_Small_US
- removed SW1: SW_Push, dylan:PTS636SK25SMTRLFS, symbol Switch:SW_Push
- removed U1: ATmega328P-AU, Package_QFP:TQFP-32_7x7mm_P0.8mm, symbol MCU_Microchip_ATmega:ATmega328P-AU
- removed VR1: LM78M05CDTX_NOPB, dylan:TO228P991X255-3N, symbol LM78M05CDTX_NOPB:LM78M05CDTX_NOPB
- removed Y1: Crystal, dylan:XTAL_ECS-160-20-5PXDN-TR, symbol Device:Crystal
- added J1: RC_PICO_Power/Coms, Connector_PinSocket_2.54mm:PinSocket_2x06_P2.54mm_Vertical_SMD, symbol Connector_Generic:Conn_02x06_Counter_Clockwise
- added J10: BackMotorOutput, Connector_PinSocket_2.54mm:PinSocket_2x06_P2.54mm_Vertical, symbol Connector:Conn_01x02_Female
- added J3: RC Reciever, Connector_PinHeader_2.54mm:PinHeader_1x04_P2.54mm_Vertical, symbol Connector:Conn_01x04_Female
- added J4: TurretServoOutput_1, Connector_PinHeader_2.54mm:PinHeader_1x03_P2.54mm_Vertical, symbol Connector:Conn_01x03_Female
- added J6: TurretServoOutput_2, Connector_PinHeader_2.54mm:PinHeader_1x03_P2.54mm_Vertical, symbol Connector:Conn_01x03_Female
- added J7: RC_PICO_Power/Coms, Connector_PinSocket_2.54mm:PinSocket_2x06_P2.54mm_Vertical, symbol Connector_Generic:Conn_02x06_Counter_Clockwise
- added J8: BackServoOutput, Connector_PinHeader_2.54mm:PinHeader_1x03_P2.54mm_Vertical, symbol Connector:Conn_01x03_Female
- added J9: FrontMotorOutput, Connector_PinSocket_2.54mm:PinSocket_2x06_P2.54mm_Vertical, symbol Connector:Conn_01x02_Female
- added U1, U2, U5, U8: Level Shifter, dylan:CONV_BOB-12009, symbol BOB-12009:BOB-12009
- added U3: RC Pico, dylan:RPi_Pico_SMD_TH, symbol MCU_RaspberryPi_and_Boards:Pico
- added U4: Autonomous Pico, dylan:RPi_Pico_SMD_TH, symbol MCU_RaspberryPi_and_Boards:Pico
- H1, H2, H3, H4: footprint MountingHole:MountingHole_2.2mm_M2 -> MountingHole:MountingHole_5.3mm_M5
- J2: value Pot -> FrontServoOutput
Connections:
- net pot is gone; now on net GND: J2.1 (Pin_1)
- net +5V: now also J1.12 (Pin_12), J3.3 (Pin_3), J7.12 (Pin_12), U1.HV, U2.HV, U3.40 (VBUS), U8.HV; no longer J2.3 (Pin_3)
- net GND: now also J1.11 (Pin_11), J1.2 (Pin_2), J10.1 (Pin_1), J3.4 (Pin_4), J4.1 (Pin_1), J6.1 (Pin_1), J7.11 (Pin_11), J7.2 (Pin_2), J8.1 (Pin_1), J9.1 (Pin_1), U1.GND_1 (GND), U1.GND_2 (GND), U2.GND_1 (GND), U2.GND_2 (GND), U3.13 (GND), U3.18 (GND), U3.23 (GND), U3.28 (GND), U3.3 (GND), U3.38 (GND), U3.42 (GND), U3.8 (GND), U4.13 (GND), U4.18 (GND), U4.23 (GND), U4.28 (GND), U4.3 (GND), U4.38 (GND), U4.42 (GND), U5.GND_1 (GND), U5.GND_2 (GND), U8.GND_1 (GND), U8.GND_2 (GND); no longer J2.2 (Pin_2)
- new net +3V3: J1.1 (Pin_1), J7.1 (Pin_1), U1.LV, U2.LV, U3.36 (3V3), U4.36 (3V3), U5.LV, U8.LV
- new net 3.3V_AUTO_BackServoSig: U4.25 (GPIO19), U5.LV2
- new net 3.3V_AUTO_FrontMotorSig: U4.21 (GPIO16)
- new net 3.3V_AUTO_FrontServoSig: U4.22 (GPIO17), U5.LV1
- new net 3.3V_AUTO_RearMotorSig: U4.24 (GPIO18)
- new net 3.3V_AUTO_WCServo1Sig: U4.11 (GPIO8), U5.LV3
- new net 3.3V_AUTO_WCServo2Sig: U4.12 (GPIO9), U5.LV4
- new net 3.3V_RC_BackServoSig: U2.LV2, U3.25 (GPIO19)
- new net 3.3V_RC_FrontMotorSig: U3.21 (GPIO16)
- new net 3.3V_RC_FrontServoSig: U2.LV1, U3.22 (GPIO17)
- new net 3.3V_RC_RearMotorSig: U3.24 (GPIO18)
- new net 3.3V_RC_WCServo1Sig: U2.LV3, U3.12 (GPIO9)
- new net 3.3V_RC_WCServo2Sig: U2.LV4, U3.11 (GPIO8)
- new net 3.3V_RX: J1.4 (Pin_4), U1.LV3, U3.7 (GPIO5)
- new net 3.3V_SCL: J1.5 (Pin_5), U1.LV2, U3.5 (GPIO3)
- new net 3.3V_SDA: J1.6 (Pin_6), U1.LV1, U3.4 (GPIO2)
- new net 3.3V_TX: J1.3 (Pin_3), U1.LV4, U3.6 (GPIO4)
- new net 5V_AUTO_BackServoSig: U5.HV2
- new net 5V_AUTO_FrontServoSig: U5.HV1
- new net 5V_AUTO_WCServo1Sig: U5.HV3
- new net 5V_AUTO_WCServo2Sig: U5.HV4
- new net 5V_RC_BackServoSig: U2.HV2
- new net 5V_RC_FrontServoSig: U2.HV1
- new net 5V_RC_WCServo1Sig: U2.HV3
- new net 5V_RC_WCServo2Sig: U2.HV4
- new net 5V_Rx: J1.8 (Pin_8), J3.1 (Pin_1), U1.HV3
- new net 5V_SCL: J1.9 (Pin_9), U1.HV2
- new net 5V_SDA: J1.10 (Pin_10), U1.HV1
- new net 5V_Tx: J1.7 (Pin_7), J3.2 (Pin_2), U1.HV4
- new net Auto_3.3V_RX: J7.4 (Pin_4), U4.6 (GPIO4), U8.LV3
- new net Auto_3.3V_SCL: J7.5 (Pin_5), U4.5 (GPIO3), U8.LV2
- new net Auto_3.3V_SDA: J7.6 (Pin_6), U4.4 (GPIO2), U8.LV1
- new net Auto_3.3V_TX: J7.3 (Pin_3), U4.7 (GPIO5), U8.LV4
- new net Auto_5V_Rx: J7.8 (Pin_8), U8.HV3
- new net Auto_5V_SCL: J7.9 (Pin_9), U8.HV2
- new net Auto_5V_SDA: J7.10 (Pin_10), U8.HV1
- new net Auto_5V_Tx: J7.7 (Pin_7), U8.HV4
- new net Auto_WaterCannonSig: U4.9 (GPIO6)
- new net BackMotorOut: J10.2 (Pin_2)
- new net BackServoOut: J8.2 (Pin_2)
- new net Battery_Voltage_ADC: U3.31 (GPIO26_ADC0), U4.31 (GPIO26_ADC0)
- new net E-Stop +5V: J2.3 (Pin_3), J4.3 (Pin_3), J6.3 (Pin_3), J8.3 (Pin_3)
- new net FrontMotorOut: J9.2 (Pin_2)
- new net FrontServoOut: J2.2 (Pin_2)
- new net RC_Auto/RC_RelaySig: U3.15 (GPIO11)
- new net RC_EStopRelaySig: U3.17 (GPIO13)
- new net RC_WaterCannonSig: U3.9 (GPIO6)
- new net TurretServoOut1: J4.2 (Pin_2)
- new net TurretServoOut2: J6.2 (Pin_2)
- no-connect marks 11 -> 40
Other:
- removed sheet RELAY
- added sheet Boat Relays (boatRelays.kicad_sch)
- added sheet Power Management (PowerManagement.kicad_sch)
- note added: "Add 5V Reg after E-Stop Switch Need to power Servos from there so it will be E-Stopped and not always powered."
- note added: "Add Voltage Dividor Circuit to read battery Voltage."
- note added: "Boat Servo/Motor Inputs"
- note added: "Need To add XT 60 for - Xavier - Router"
- note added: "Need to figure out best way to wire up Physical E-Stop Button, what type of connector to the board?"
- note added: "Water Cannon Servo Turrent Inputs"
- note added: "What type of connector should the water pump plug into the board as?"
- moved on the sheet: D5, D6, D7, H1, H2, H3, H4, J2, J5, R6, R7, R8
